Commit message: Update simple_robot.urdf

File: simple_robot.urdf (robot description, URDF)
Before this commit: robot simple_robot, 3 links, 2 joints
Links:
- added link link3; visual cylinder length=0.2 radius=0.04
Joints:
- added joint joint3: type revolute, parent link2, child link3, origin xyz=0.3 0 0, axis 0 -1 0, limit lower=-3.14 upper=3.14 effort=300 velocity=0.1
